File: Control_Board/Control_Board.kicad_pcb (KiCad board)
At the start: 4 copper layers, 87 x 105 mm, 85 parts, among them J1 Barrel_Jack_Switch, J2 C2982037, J3 C2982037, J4 C2982037, J5 C2982037, P0 MOLEX 530470410, P1 MOLEX 530470410, P2 MOLEX 530470410, P3 MOLEX 530470410, P4 MOLEX 530470410, P5 MOLEX 530470410, P6 MOLEX 530470410, P7 MOLEX 530470410, Q0 MOLEX 530470610, Q1 MOLEX 530470610, Q2 MOLEX 530470610, Q3 MOLEX 530470610, Q4 MOLEX 530470610, Q5 MOLEX 530470610, Q6 MOLEX 530470610, Q7 MOLEX 530470610, Q8 AO3407A, U1 TLV76133DCY, U2 AZ1084CD-5.0TRG1, U3 TCA9406DCUR

Commit message: Folders cleaned
Other:
- board text added: "EvolChip Control Board Charité - Labor für Biofluidmechanik Input: 9V - 2A Version: 1.0"
- board text removed: "EvolChip Evaluation Board Charité - Labor für Biofluidmechanik Input: 9V - 2A Version: 1.0"
