File: Honeywell_HSC_Pressure_Sensor/Honeywell_HSC_SMT.kicad_pcb (KiCad board)
At the start: 2 copper layers, 20 x 22 mm, 6 parts, among them J1 Conn_01x04

Commit message: Honeywell_HSC_Pressure_Sensor break out board: changed 4.7kOhm to 10kOhm
Parts:
- R1, R2: value 4.7k -> 10k
Other:
- board text added: "Honeywell HSC Pressure Sensor 1 psi VDD: 3.3V"
- board text removed: "Honeywell HSC SMT Pressure Sensor 1 psi VDD: 3.3V"
Changed lines of the file:
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@@
 			)
 		)
-		(property "Value" "4.7k"
+		(property "Value" "10k"
 			(at 0 1.43 0)
 			(layer "F.Fab")
@@
 			)
 		)
-		(property "Value" "4.7k"
+		(property "Value" "10k"
 			(at 0 1.43 0)
 			(layer "F.Fab")
@@
 		)
 	)
-	(gr_text "Honeywell HSC SMT\nPressure Sensor\n1 psi\nVDD: 3.3V"
+	(gr_text "Honeywell HSC\nPressure Sensor\n1 psi\nVDD: 3.3V"
 		(at 22.08 20.87 0)
 		(layer "B.SilkS" knockout)
